File: !Kursach/Arduino_MEGA_START/Arduino_MEGA_2560-Rev3.kicad_pcb (KiCad board)
At the start: 2 copper layers, 101.6 x 53.3 mm, 6 parts

Commit message: c
Parts:
- added D1: Drive_Connector, Connector_PinHeader_2.54mm:PinHeader_1x02_P2.54mm_Vertical, F.Cu at (188.6, 86.0)
- added D10: Drive_Connector, Connector_PinHeader_2.54mm:PinHeader_1x02_P2.54mm_Vertical, F.Cu at (263.5, 58.9)
- added D11: Drive_Connector, Connector_PinHeader_2.54mm:PinHeader_1x02_P2.54mm_Vertical, F.Cu at (248.5, 103.8)
- added D12: Drive_Connector, Connector_PinHeader_2.54mm:PinHeader_1x02_P2.54mm_Vertical, F.Cu at (246.8, 80.3)
- added D13: Drive_Connector, Connector_PinHeader_2.54mm:PinHeader_1x02_P2.54mm_Vertical, F.Cu at (263.5, 69.6)
- added D14: Drive_Connector, Connector_PinHeader_2.54mm:PinHeader_1x02_P2.54mm_Vertical, F.Cu at (280.2, 58.9)
- added D15: Drive_Connector, Connector_PinHeader_2.54mm:PinHeader_1x02_P2.54mm_Vertical, F.Cu at (188.7, 116.5)
- added D16: Drive_Connector, Connector_PinHeader_2.54mm:PinHeader_1x02_P2.54mm_Vertical, F.Cu at (120.7, 102.0)
- added D17: Drive_Connector, Connector_PinHeader_2.54mm:PinHeader_1x02_P2.54mm_Vertical, F.Cu at (137.3, 91.3)
- added D18: Drive_Connector, Connector_PinHeader_2.54mm:PinHeader_1x02_P2.54mm_Vertical, F.Cu at (120.7, 91.3)
- added D2: Drive_Connector, Connector_PinHeader_2.54mm:PinHeader_1x02_P2.54mm_Vertical, F.Cu at (188.7, 91.1)
- added D3: Drive_Connector, Connector_PinHeader_2.54mm:PinHeader_1x02_P2.54mm_Vertical, F.Cu at (188.7, 96.1)
- added D4: Drive_Connector, Connector_PinHeader_2.54mm:PinHeader_1x02_P2.54mm_Vertical, F.Cu at (188.7, 101.2)
- added D5: Drive_Connector, Connector_PinHeader_2.54mm:PinHeader_1x02_P2.54mm_Vertical, F.Cu at (188.7, 106.3)
- added D6: Drive_Connector, Connector_PinHeader_2.54mm:PinHeader_1x02_P2.54mm_Vertical, F.Cu at (188.7, 111.4)
- added D7: Drive_Connector, Connector_PinHeader_2.54mm:PinHeader_1x02_P2.54mm_Vertical, F.Cu at (254.1, 107.8)
- added D8: Drive_Connector, Connector_PinHeader_2.54mm:PinHeader_1x02_P2.54mm_Vertical, F.Cu at (188.7, 121.5)
- added D9: Drive_Connector, Connector_PinHeader_2.54mm:PinHeader_1x02_P2.54mm_Vertical, F.Cu at (246.8, 69.6)
- added J1: RX, Connector_PinHeader_2.54mm:PinHeader_1x02_P2.54mm_Vertical, F.Cu at (163.6, 83.3)
- added J2: TX, Connector_PinHeader_2.54mm:PinHeader_1x02_P2.54mm_Vertical, F.Cu at (161.0, 83.3)
- added PWMH1: 8x1F-H8.5, Connector_PinHeader_2.54mm:PinHeader_1x08_P2.54mm_Vertical, F.Cu at (138.7, 80.8)
Connections:
- net /GND renamed GND
- PWML1 pad 3: /PE4 -> /Dir17
- PWML1 pad 5: /PG5 -> /Dir18
- XIO1 pad 1: /+5V -> Net-(XIO1-Pad1)
- XIO1 pad 10: /PA7 -> /P29
- XIO1 pad 11: /PC7 -> /Dir3
- XIO1 pad 12: /PC6 -> /Dir11
- XIO1 pad 13: /PC5 -> /P32
- XIO1 pad 14: /PC4 -> /P33
- XIO1 pad 15: /PC3 -> /Dir4
- XIO1 pad 16: /PC2 -> /Dir12
- XIO1 pad 17: /PC1 -> /P36
- XIO1 pad 18: /PC0 -> /P37
- XIO1 pad 19: /PD7 -> /Dir5
- XIO1 pad 2: /+5V -> Net-(XIO1-Pad2)
- XIO1 pad 20: /PG2 -> /Dir13
- XIO1 pad 21: /PG1 -> /P40
- XIO1 pad 22: /PG0 -> /P41
- XIO1 pad 23: /PL7 -> /Dir6
- XIO1 pad 24: /PL6 -> /Dir14
- XIO1 pad 25: /PL5 -> /P44
- XIO1 pad 26: /PL4 -> /P45
- XIO1 pad 27: /PL3 -> /Dir7
- XIO1 pad 28: /PL2 -> /Dir15
- XIO1 pad 29: /PL1 -> /P48
- XIO1 pad 3: /PA0 -> /Dir1
- XIO1 pad 30: /PL0 -> /P49
- XIO1 pad 31: /PB3 -> /Dir8
- XIO1 pad 32: /PB2 -> /Dir16
- XIO1 pad 33: /PB1 -> /P52
- XIO1 pad 34: /PB0 -> /P53
- XIO1 pad 4: /PA1 -> /Dir9
- XIO1 pad 5: /PA2 -> /P24
- XIO1 pad 6: /PA3 -> /P25
- XIO1 pad 7: /PA4 -> /Dir2
- XIO1 pad 8: /PA5 -> /Dir10
- XIO1 pad 9: /PA6 -> /P28
Other:
- board size 101.6 x 53.3 mm -> 85 x 53.3 mm

Commit message: S
Parts:
- added J3: Midi_UART, Connector_PinHeader_2.54mm:PinHeader_1x03_P2.54mm_Vertical, F.Cu at (167.1, 88.5)
- added J4: USB_Uart, Connector_PinHeader_2.54mm:PinHeader_1x03_P2.54mm_Vertical, F.Cu at (176.5, 88.4)
- added J5: Power_conn, Connector_PinHeader_2.54mm:PinHeader_1x02_P2.54mm_Vertical, F.Cu at (140.8, 125.0)
- moved D14 97.1 mm to (198.8, 111.9), turned to 180 degrees
- moved D18 84.0 mm to (198.8, 122.3), turned to 180 degrees
- moved D13 74.6 mm to (198.8, 106.7), turned to 180 degrees
- moved D10 72.3 mm to (198.8, 91.1), turned to 180 degrees
- moved D7 68.1 mm to (186.7, 117.5), turned to 180 degrees
- moved D12 52.5 mm to (198.8, 101.5), turned to 180 degrees
- moved D9 50.7 mm to (198.8, 85.9), turned to 180 degrees
- moved D11 50.3 mm to (198.8, 96.5), turned to 180 degrees
- moved D16 36.6 mm to (154.7, 88.5), turned to 90 degrees
- moved D17 11.6 mm to (148.6, 88.4), turned to 90 degrees
- moved D15 10.1 mm to (198.8, 117.1)
- moved D4 2.33 mm to (186.6, 102.1)
- moved D5 2.33 mm to (186.6, 107.2)
- moved D6 2.33 mm to (186.6, 112.3)
- moved D8 2.22 mm to (186.7, 122.4)
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Connections:
- net /Led3 renamed Net-(J1-Pad1)
- net /Led4 renamed Net-(J2-Pad1)
Other:
- board size 85 x 53.3 mm -> 100.7 x 53.4 mm

Commit message: s
Parts:
- added C1: 22pF, Capacitor_SMD:C_1206_3216Metric_Pad1.33x1.80mm_HandSolder, F.Cu at (134.0, 94.2)
- added C2: 22pF, Capacitor_SMD:C_1206_3216Metric_Pad1.33x1.80mm_HandSolder, F.Cu at (118.9, 94.2)
- added C3: 10uF, Capacitor_Tantalum_SMD:CP_EIA-6032-15_Kemet-U_Pad2.25x2.35mm_HandSolder, F.Cu at (139.7, 95.6)
- added D19: Drive_Connector, Connector_PinHeader_2.54mm:PinHeader_1x02_P2.54mm_Vertical, F.Cu at (142.5, 88.5)
- added D20: Drive_Connector, Connector_PinHeader_2.54mm:PinHeader_1x02_P2.54mm_Vertical, F.Cu at (130.8, 85.0)
- added D21: Drive_Connector, Connector_PinHeader_2.54mm:PinHeader_1x02_P2.54mm_Vertical, F.Cu at (137.3, 85.0)
- added D22: Drive_Connector, Connector_PinHeader_2.54mm:PinHeader_1x02_P2.54mm_Vertical, F.Cu at (124.5, 85.0)
- added D23: Drive_Connector, Connector_PinHeader_2.54mm:PinHeader_1x02_P2.54mm_Vertical, F.Cu at (156.1, 125.3)
- added D24: Drive_Connector, Connector_PinHeader_2.54mm:PinHeader_1x02_P2.54mm_Vertical, F.Cu at (150.6, 125.3)
- added D25: Drive_Connector, Connector_PinHeader_2.54mm:PinHeader_1x02_P2.54mm_Vertical, F.Cu at (161.7, 125.3)
- added D26: Drive_Connector, Connector_PinHeader_2.54mm:PinHeader_1x02_P2.54mm_Vertical, F.Cu at (171.3, 125.3)
- added D27: Drive_Connector, Connector_PinHeader_2.54mm:PinHeader_1x02_P2.54mm_Vertical, F.Cu at (164.8, 125.3)
- added D28: Drive_Connector, Connector_PinHeader_2.54mm:PinHeader_1x02_P2.54mm_Vertical, F.Cu at (176.8, 125.3)
- added D29: Drive_Connector, Connector_PinHeader_2.54mm:PinHeader_1x02_P2.54mm_Vertical, F.Cu at (179.6, 121.2)
- added D30: Drive_Connector, Connector_PinHeader_2.54mm:PinHeader_1x02_P2.54mm_Vertical, F.Cu at (186.6, 126.0)
- added Di1: 3.6V, Diode_THT:D_DO-41_SOD81_P7.62mm_Horizontal, F.Cu at (131.2, 116.7)
- added Di2: 3.6V, Diode_THT:D_DO-41_SOD81_P7.62mm_Horizontal, F.Cu at (131.2, 113.3)
- added J6: USB, usb_type_c_female_board_Aliexpress:usb_type_c_female_board_Aliexpress, F.Cu at (115.1, 115.6)
- added J7: Usb_ext, Connector_PinSocket_2.54mm:PinSocket_1x04_P2.54mm_Vertical, F.Cu at (116.1, 105.5)
- added R1: 68, Resistor_THT:R_Axial_DIN0204_L3.6mm_D1.6mm_P2.54mm_Vertical, F.Cu at (125.3, 116.5)
- added R2: 68, Resistor_THT:R_Axial_DIN0204_L3.6mm_D1.6mm_P2.54mm_Vertical, F.Cu at (125.3, 113.4)
- added R3: 2.2k, Resistor_THT:R_Axial_DIN0204_L3.6mm_D1.6mm_P2.54mm_Vertical, F.Cu at (125.1, 124.2)
- added U1: ATmega8A-PU, Package_DIP:DIP-28_W7.62mm, F.Cu at (168.3, 101.0)
- added Y1: 16M, Crystal:Crystal_HC49-4H_Vertical, F.Cu at (124.0, 94.6)
- moved J1 0.38 mm to (140.8, 125.3)
- moved J3 0.25 mm to (161.0, 83.6)
- moved D17 0.13 mm to (148.6, 88.5)
- moved J2 0.13 mm to (163.7, 83.3)
- moved J4 0.13 mm to (167.1, 88.4)
- renumbered D2 to D1, D11 to D10, D12 to D11, D13 to D12, D14 to D13, D15 to D14, D1 to D15, D18 to D16, D16 to D18, D3 to D2, D4 to D3, D5 to D4, D6 to D5, D7 to D6, D8 to D7, D9 to D8, D10 to D9, J5 to J1, J1 to J2, J2 to J3, J3 to J4, J4 to J5
Connections:
- PWMH1 pad 1: /PH5 -> /Dir20
- PWMH1 pad 3: /PB4 -> /Dir21
- PWMH1 pad 5: /PB6 -> /Dir22
- PWML1 pad 7: /PH3 -> /Dir19
Other:
- outline, holes or cut-outs redrawn
- board text added: "23"
- board text added: "25"
- board text added: "27"
