File: !Kursach/Arduino_MEGA_START/Arduino_MEGA_2560-Rev3.sch (KiCad schematic (older format))
At the start: 6 parts

Commit message: c
Parts:
- added J1: RX, Connector_PinHeader_2.54mm:PinHeader_1x02_P2.54mm_Vertical, symbol Connector:Conn_01x02_Male
- added J2: TX, Connector_PinHeader_2.54mm:PinHeader_1x02_P2.54mm_Vertical, symbol Connector:Conn_01x02_Male
- added PWMH1: 8x1F-H8.5, Connector_PinHeader_2.54mm:PinHeader_1x08_P2.54mm_Vertical, symbol Arduino_MEGA_2560-Rev3:SMARTPRJ_PINHD-1X8
Connections:
- net +5V: no longer XIO1.1, XIO1.2
- net GND: now also PWMH1.7
- net PE0: now also J1.2 (Pin_2)
- net PE1: now also J2.2 (Pin_2)
- net PA0 renamed Dir1
- net PA1 renamed Dir9
- net PA2 renamed P24
- net PA3 renamed P25
- net PA4 renamed Dir2
- net PA5 renamed Dir10
- net PA6 renamed P28
- net PA7 renamed P29
- net PB0 renamed P53
- net PB1 renamed P52
- net PB2 renamed Dir16
- net PB3 renamed Dir8
- net PC0 renamed P37
- net PC1 renamed P36
- net PC2 renamed Dir12
- net PC3 renamed Dir4
- net PC4 renamed P33
- net PC5 renamed P32
- net PC6 renamed Dir11
- net PC7 renamed Dir3
- net PD7 renamed Dir5
- net PE4 renamed Dir17
- net PG0 renamed P41
- net PG1 renamed P40
- net PG2 renamed Dir13
- net PG5 renamed Dir18
- net PL0 renamed P49
- net PL1 renamed P48
- net PL2 renamed Dir15
- net PL3 renamed Dir7
- net PL4 renamed P45
- net PL5 renamed P44
- net PL6 renamed Dir14
- net PL7 renamed Dir6
- new net Aref: PWMH1.8
- new net Led3: J1.1 (Pin_1)
- new net Led4: J2.1 (Pin_1)
- new net PB4: PWMH1.3
- new net PB5: PWMH1.4
- new net PB6: PWMH1.5
- new net PB7: PWMH1.6
- new net PH5: PWMH1.1
- new net PH6: PWMH1.2
- no-connect marks 0 -> 3
Other:
- note added: "10"
- note added: "11"
- note added: "12"
- note added: "13"
- note added: "8"
- note added: "9\n"
- note added: "AREF"
- moved on the sheet: ADCH1, ADCL1, COMMUNICATION1, POWER1, PWML1, XIO1

Commit message: S
Parts:
- added J3: Midi_UART, Connector_PinHeader_2.54mm:PinHeader_1x03_P2.54mm_Vertical, symbol Connector:Conn_01x03_Male
- added J4: USB_Uart, Connector_PinHeader_2.54mm:PinHeader_1x03_P2.54mm_Vertical, symbol Connector:Conn_01x03_Male
- added J5: Power_conn, Connector_PinHeader_2.54mm:PinHeader_1x02_P2.54mm_Vertical, symbol Connector:Conn_01x02_Male
- added U?: 74HCT595, symbol 74xx:74HCT595
Connections:
- net GND: now also J3.1 (Pin_1), J4.1 (Pin_1), J5.1 (Pin_1)
- net RXD2: now also J4.2 (Pin_2)
- net RXD3: now also J3.2 (Pin_2)
- net TXD2: now also J4.3 (Pin_3)
- net TXD3: now also J3.3 (Pin_3)
- net VIN: now also J5.2 (Pin_2)
- net Led3: no longer names the net of J1.1 (Pin_1)
- net Led4: no longer names the net of J2.1 (Pin_1)
- no-connect marks 3 -> 5
Changed lines of the file:
@@
 U 1 1 5A5FE3D3
 P 6700 3050
-F 0 "COMMUNICATION1" H 7075 3050 70  0000 L BNN
+F 0 "COMMUNICATION1" H 6450 2400 70  0000 L BNN
 F 1 "8x1F-H8.5" H 6451 2550 70  0000 L BNN
 F 2 "Arduino_MEGA_2560-Rev3:SMARTPRJ_1X08" H 6690 2840 65  0001 L TNN
@@
 Wire Wire Line
 	7350 4250 6600 4250
-Text Label 7550 4250 0    50   ~ 0
-Led4
-Wire Wire Line
-	7450 4250 7550 4250
 Wire Wire Line
 	6900 4150 6600 4150
@@
 Wire Wire Line
 	1600 9500 1700 9500
-Text Label 7250 4550 0    50   ~ 0
-Led3
 $Sheet
 S 2700 9500 500  350
@@
 Text Label 6900 3850 0    50   ~ 0
 Step18
+NoConn ~ 7450 4250
+NoConn ~ 7250 4550
+$Comp
+L Connector:Conn_01x03_Male J3
+U 1 1 61469229
+P 7550 2750
+F 0 "J3" H 7522 2682 50  0000 R CNN
+F 1 "Midi_UART" H 7522 2773 50  0000 R CNN
+F 2 "Connector_PinHeader_2.54mm:PinHeader_1x03_P2.54mm_Vertical" H 7550 2750 50  0001 C CNN
+F 3 "~" H 7550 2750 50  0001 C CNN
+	1    7550 2750
+	-1   0    0    1
+$EndComp
+$Comp
+L Connector:Conn_01x03_Male J4
+U 1 1 6146FE40
+P 7550 3100
+F 0 "J4" H 7522 3032 50  0000 R CNN
+F 1 "USB_Uart" H 7522 3123 50  0000 R CNN
+F 2 "Connector_PinHeader_2.54mm:PinHeader_1x03_P2.54mm_Vertical" H 7550 3100 50  0001 C CNN
+F 3 "~" H 7550 3100 50  0001 C CNN
+	1    7550 3100
+	-1   0    0    1
+$EndComp
+Text Label 7300 2650 2    10   ~ 0
+TXD3
+Text Label 7300 2750 2    10   ~ 0
+RXD3
+Text Label 7300 3000 2    10   ~ 0
+TXD2
+Text Label 7300 3100 2    10   ~ 0
+RXD2
+Wire Wire Line
+	7350 2650 7300 2650
+Wire Wire Line
+	7350 2750 7300 2750
+Wire Wire Line
+	7350 3000 7300 3000
+Wire Wire Line
+	7350 3100 7300 3100
+$Comp
+L power:GND #PWR0101
+U 1 1 6148674B
+P 7300 3300
+F 0 "#PWR0101" H 7300 3050 50  0001 C CNN
+F 1 "GND" H 7450 3300 50  0000 C CNN
+F 2 "" H 7300 3300 50  0001 C CNN
+F 3 "" H 7300 3300 50  0001 C CNN
+	1    7300 3300
+	1    0    0    -1
+$EndComp
+Wire Wire Line
+	7300 3300 7300 3200
+Wire Wire Line
+	7300 3200 7350 3200
+$Comp
+L power:GND #PWR0102
+U 1 1 6148EAB9
+P 7200 2900
+F 0 "#PWR0102" H 7200 2650 50  0001 C CNN
+F 1 "GND" H 7100 2900 50  0000 C CNN
+F 2 "" H 7200 2900 50  0001 C CNN
+F 3 "" H 7200 2900 50  0001 C CNN
+	1    7200 2900
+	1    0    0    -1
+$EndComp
+Wire Wire Line
+	7200 2900 7200 2850
+Wire Wire Line
+	7200 2850 7350 2850
+$Comp
+L Connector:Conn_01x02_Male J5
+U 1 1 6149D75C
+P 5100 3350
+F 0 "J5" H 5208 3531 50  0000 C CNN
+F 1 "Power_conn" H 5208 3440 50  0000 C CNN
+F 2 "Connector_PinHeader_2.54mm:PinHeader_1x02_P2.54mm_Vertical" H 5100 3350 50  0001 C CNN
+F 3 "~" H 5100 3350 50  0001 C CNN
+	1    5100 3350
+	1    0    0    -1
+$EndComp
+Wire Wire Line
+	5300 3350 5550 3350
+Connection ~ 5550 3350
+Wire Wire Line
+	5300 3450 5550 3450
+$Comp
+L 74xx:74HCT595 U?
+U 1 1 614AB632
+P 7950 8250
+F 0 "U?" H 7950 9031 50  0000 C CNN
+F 1 "74HCT595" H 7950 8940 50  0000 C CNN
+F 2 "" H 7950 8250 50  0001 C CNN
+F 3 "https://assets.nexperia.com/documents/data-sheet/74HC_HCT595.pdf" H 7950 8250 50  0001 C CNN
+	1    7950 8250
+	1    0    0    -1
+$EndComp
 $EndSCHEMATC

Commit message: s
Parts:
- removed U?: 74HCT595, symbol 74xx:74HCT595
- added C1, C2: 22pF, Capacitor_SMD:C_1206_3216Metric_Pad1.33x1.80mm_HandSolder, symbol Device:C_Small
- added C3: 10uF, Capacitor_Tantalum_SMD:CP_EIA-6032-15_Kemet-U_Pad2.25x2.35mm_HandSolder, symbol Device:C_Small
- added Di1, Di2: 3.6V, Diode_THT:D_DO-41_SOD81_P7.62mm_Horizontal, symbol Device:D_Zener_Small
- added J6: USB, usb_type_c_female_board_Aliexpress:usb_type_c_female_board_Aliexpress, symbol Connector:Conn_01x04_Female
- added J7: Usb_ext, Connector_PinSocket_2.54mm:PinSocket_1x04_P2.54mm_Vertical, symbol Connector:Conn_01x04_Male
- added R1, R2: 68, Resistor_THT:R_Axial_DIN0204_L3.6mm_D1.6mm_P2.54mm_Vertical, symbol Device:R_Small
- added R3: 2.2k, Resistor_THT:R_Axial_DIN0204_L3.6mm_D1.6mm_P2.54mm_Vertical, symbol Device:R_Small
- added U1: ATmega8A-PU, Package_DIP:DIP-28_W7.62mm, symbol MCU_Microchip_ATmega:ATmega8A-PU
- added Y1: 16M, Crystal:Crystal_HC49-4H_Vertical, symbol Device:Crystal
- renumbered J5 to J1, J1 to J2, J2 to J3, J3 to J4, J4 to J5
Connections:
- net GND: now also C1.1, C2.1, C3.2, Di1.2 (A), Di2.2 (A), J6.4 (Pin_4), J7.4 (Pin_4), U1.8 (GND)
- net RXD2: now also U1.3 (PD1)
- net TXD2: now also U1.2 (PD0)
- net PB4 renamed Dir21
- net PB6 renamed Dir22
- net PH3 renamed Dir19
- net PH5 renamed Dir20
- new net: J6.2 (Pin_2), J7.2 (Pin_2), R1.1
- new net: J6.3 (Pin_3), J7.3 (Pin_3), R2.1
- new net: C2.2, U1.10 (PB7/XTAL2), Y1.1
- new net: C1.2, U1.9 (PB6/XTAL1), Y1.2
- new net D+: Di2.1 (K), R2.2, U1.4 (PD2)
- new net D-: Di1.1 (K), R1.2, R3.2, U1.5 (PD3)
- new net U_pull_up: U1.6 (PD4)
- new net U_vcc: C3.1, J6.1 (Pin_1), J7.1 (Pin_1), R3.1, U1.7 (VCC)
- no-connect marks 5 -> 24
Other:
- note added: "D+"
- note added: "D-"
- note added: "U_Gnd"
- note added: "Usb 5v"
