File: !Kursach/Arduino_MEGA_START/drive_conn.sch (KiCad schematic (older format))
At the start: 1 part

Commit message: S
Changed lines of the file:
@@
 $Descr A4 11693 8268
 encoding utf-8
-Sheet 8 19
+Sheet 17 19
 Title ""
 Date ""
@@
 AR Path="/614769B2/6143D9DF" Ref="D16"  Part="1"
 AR Path="/6147D787/6143D9DF" Ref="D17"  Part="1"
-F 0 "D8" H 2122 1582 50  0000 R CNN
+F 0 "D16" H 2122 1582 50  0000 R CNN
 F 1 "Drive_Connector" H 2122 1673 50  0000 R CNN
 F 2 "Connector_PinHeader_2.54mm:PinHeader_1x02_P2.54mm_Vertical" H 2150 1700 50  0001 C CNN

Commit message: s
Parts:
- renumbered D1 to D15
Changed lines of the file:
@@
 $Descr A4 11693 8268
 encoding utf-8
-Sheet 17 19
+Sheet 17 31
 Title ""
 Date ""
@@
 	1950 1700 1750 1700
 $Comp
-L Connector:Conn_01x02_Male D1
+L Connector:Conn_01x02_Male D15
 U 1 1 6143D9DF
 P 2150 1700
-AR Path="/61428437/6143D9DF" Ref="D1"  Part="1"
-AR Path="/6146C0B8/6143D9DF" Ref="D2"  Part="1"
-AR Path="/6146D738/6143D9DF" Ref="D3"  Part="1"
-AR Path="/614718A7/6143D9DF" Ref="D4"  Part="1"
-AR Path="/614718B2/6143D9DF" Ref="D5"  Part="1"
-AR Path="/614718BD/6143D9DF" Ref="D6"  Part="1"
-AR Path="/61473FF9/6143D9DF" Ref="D7"  Part="1"
-AR Path="/61474004/6143D9DF" Ref="D8"  Part="1"
-AR Path="/6147DE01/6143D9DF" Ref="D9"  Part="1"
-AR Path="/614810D6/6143D9DF" Ref="D10"  Part="1"
-AR Path="/614810E0/6143D9DF" Ref="D11"  Part="1"
-AR Path="/614810EA/6143D9DF" Ref="D12"  Part="1"
-AR Path="/6148D253/6143D9DF" Ref="D13"  Part="1"
-AR Path="/6148D25D/6143D9DF" Ref="D14"  Part="1"
-AR Path="/6148D267/6143D9DF" Ref="D15"  Part="1"
-AR Path="/61462287/6143D9DF" Ref="D18"  Part="1"
-AR Path="/614769B2/6143D9DF" Ref="D16"  Part="1"
+AR Path="/61428437/6143D9DF" Ref="D15"  Part="1"
+AR Path="/6146C0B8/6143D9DF" Ref="D1"  Part="1"
+AR Path="/6146D738/6143D9DF" Ref="D2"  Part="1"
+AR Path="/614718A7/6143D9DF" Ref="D3"  Part="1"
+AR Path="/614718B2/6143D9DF" Ref="D4"  Part="1"
+AR Path="/614718BD/6143D9DF" Ref="D5"  Part="1"
+AR Path="/61473FF9/6143D9DF" Ref="D6"  Part="1"
+AR Path="/61474004/6143D9DF" Ref="D7"  Part="1"
+AR Path="/6147DE01/6143D9DF" Ref="D8"  Part="1"
+AR Path="/614810D6/6143D9DF" Ref="D9"  Part="1"
+AR Path="/614810E0/6143D9DF" Ref="D10"  Part="1"
+AR Path="/614810EA/6143D9DF" Ref="D11"  Part="1"
+AR Path="/6148D253/6143D9DF" Ref="D12"  Part="1"
+AR Path="/6148D25D/6143D9DF" Ref="D13"  Part="1"
+AR Path="/6148D267/6143D9DF" Ref="D14"  Part="1"
+AR Path="/61462287/6143D9DF" Ref="D16"  Part="1"
+AR Path="/614769B2/6143D9DF" Ref="D18"  Part="1"
 AR Path="/6147D787/6143D9DF" Ref="D17"  Part="1"
-F 0 "D16" H 2122 1582 50  0000 R CNN
+AR Path="/61847DBB/6143D9DF" Ref="D?"  Part="1"
+AR Path="/61849843/6143D9DF" Ref="D19"  Part="1"
+AR Path="/61853C76/6143D9DF" Ref="D20"  Part="1"
+AR Path="/61853C7C/6143D9DF" Ref="D21"  Part="1"
+AR Path="/61853C84/6143D9DF" Ref="D22"  Part="1"
+AR Path="/618BA597/6143D9DF" Ref="D23"  Part="1"
+AR Path="/618BA59D/6143D9DF" Ref="D24"  Part="1"
+AR Path="/618BA5A4/6143D9DF" Ref="D25"  Part="1"
+AR Path="/618FBCF1/6143D9DF" Ref="D26"  Part="1"
+AR Path="/618FBCF7/6143D9DF" Ref="D27"  Part="1"
+AR Path="/618FBCFE/6143D9DF" Ref="D28"  Part="1"
+AR Path="/6193E98E/6143D9DF" Ref="D29"  Part="1"
+AR Path="/6193E995/6143D9DF" Ref="D30"  Part="1"
+F 0 "D30" H 2122 1582 50  0000 R CNN
 F 1 "Drive_Connector" H 2122 1673 50  0000 R CNN
 F 2 "Connector_PinHeader_2.54mm:PinHeader_1x02_P2.54mm_Vertical" H 2150 1700 50  0001 C CNN
