File: !Kursach/LX/lx_ind/555+mt3608.sch (KiCad schematic (older format))
At the start: 38 parts, among them J1 Bat, Q1 2N7002E, SW1 SW_Push, U1 SA555D, U2 LM317L_TO92, U3 LM358, U4 LM339

Commit message: s
Parts:
- added C4, C5: 10uF, Capacitor_SMD:C_1206_3216Metric_Pad1.33x1.80mm_HandSolder, symbol Device:C_Small
- added C6: 100uF, Capacitor_THT:CP_Radial_D10.0mm_P5.00mm, symbol Device:CP_Small
- added D6: SS34, Diode_SMD:D_SMC, symbol Device:D_Schottky_Small
- added J2: Bat, Connector_PinSocket_2.54mm:PinSocket_1x02_P2.54mm_Horizontal, symbol Connector:Conn_01x02_Male
- added J3: Bat_en, Connector_PinSocket_2.54mm:PinSocket_1x02_P2.54mm_Horizontal, symbol Connector:Conn_01x02_Male
- added J4: V_Out, Connector_PinSocket_2.54mm:PinSocket_1x02_P2.54mm_Horizontal, symbol Connector:Conn_01x02_Male
- added L1: 22uH, Inductor_SMD:L_Bourns_SRR1210A, symbol Device:L
- added R20: 2.2k, Resistor_SMD:R_1206_3216Metric_Pad1.30x1.75mm_HandSolder, symbol Device:R_Small
- added RV5: 100k, Potentiometer_SMD:Potentiometer_Bourns_TC33X_Vertical, symbol Device:R_POT_Small
- added U5: MT3608, Package_TO_SOT_SMD:SOT-23-6_Handsoldering, symbol Regulator_Switching:MT3608
- C1, C3: footprint (none) -> Capacitor_SMD:C_1206_3216Metric_Pad1.33x1.80mm_HandSolder
- C2: footprint (none) -> Capacitor_Tantalum_SMD:CP_EIA-3216-10_Kemet-I_Pad1.58x1.35mm_HandSolder
- D1, D2, D3, D4, D5: footprint (none) -> LED_SMD:LED_1206_3216Metric_Pad1.42x1.75mm_HandSolder
- J1: value Bat -> Bat_in; footprint (none) -> Connector_PinSocket_2.54mm:PinSocket_1x02_P2.54mm_Horizontal
- Q1: value 2N7002E -> SSM3K333R,LF
- R1, R10, R11, R12, R13, R14, R15, R16, R17, R18, R19, R2, R3, R4, R5, R6, R7, R8, R9: footprint (none) -> Resistor_SMD:R_1206_3216Metric_Pad1.30x1.75mm_HandSolder
- RV1, RV2, RV3, RV4: footprint (none) -> Potentiometer_SMD:Potentiometer_Bourns_TC33X_Vertical
- SW1: footprint (none) -> Button_Switch_SMD:SW_SPST_EVPBF
- U3: footprint (none) -> Package_SO:SO-8_3.9x4.9mm_P1.27mm
- U4: footprint (none) -> Package_SO:SO-14_3.9x8.65mm_P1.27mm
Connections:
- net GND: now also C4.2, C5.2, C6.2, J2.2 (Pin_2), J4.1 (Pin_1), R20.2, U5.2 (GND)
- net at C3.1, D1.2 (A), D2.2 (A)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: no longer R14.1, R15.2, U4.2
- net Bat_in: now reaches J1.1 (Pin_1), Q1.3 (D), R1.1, R3.2, U1.8 (VCC)
- net Bat_in: now also C4.1, J3.1 (Pin_1), L1.1, U5.4 (EN), U5.5 (IN)
- new net: R14.1, R15.2, U4.2
- new net: J2.1 (Pin_1), J3.2 (Pin_2)
- new net: R20.1, RV5.1
- new net: RV5.2, U5.3 (FB)
- new net: D6.2 (A), L1.2, U5.1 (SW)
- new net Vout_12V: C5.1, C6.1, D6.1 (K), J4.2 (Pin_2), RV5.3
Other:
- note added: "какой найдем на самом делу"
- moved on the sheet: J1
