File: !Kursach/DMK/dml/dml.sch (KiCad schematic (older format))
At the start: 26 parts, among them J1 Debug, J2 Conn_01x01_Male, J3 USB, SW1 SW_Push, SW2 SW_Push, U1 HEF4093B

Commit message: s
Parts:
- removed C3: 0.1uF, Capacitor_SMD:C_0805_2012Metric_Pad1.18x1.45mm_HandSolder, symbol Device:C_Small
- removed D3, D4: WS2812B, LED_SMD:LED_WS2812B_PLCC4_5.0x5.0mm_P3.2mm, symbol LED:WS2812B
- removed J1: Debug, Connector_PinSocket_2.54mm:PinSocket_1x02_P2.54mm_Vertical, symbol Connector:Conn_01x02_Male
- removed R6: 2.2k, Resistor_THT:R_Axial_DIN0204_L3.6mm_D1.6mm_P2.54mm_Vertical, symbol Device:R_Small
- added C4, C5: 100nF???10nF, Capacitor_SMD:C_0805_2012Metric_Pad1.18x1.45mm_HandSolder, symbol Device:C_Small
- added J3, J4: Conn_01x01_Male, Connector_PinHeader_2.54mm:PinHeader_1x01_P2.54mm_Vertical, symbol Connector:Conn_01x01_Male
- added J5, J6: Conn_01x01_Female, Connector_PinHeader_2.54mm:PinHeader_1x01_P2.54mm_Vertical, symbol Connector:Conn_01x01_Female
- added J7: Conn_01x04_Male, Connector_PinHeader_2.54mm:PinHeader_1x04_P2.54mm_Vertical, symbol Connector:Conn_01x04_Male
- added J8: Conn_01x04_Female, Connector_PinHeader_2.54mm:PinHeader_1x04_P2.54mm_Vertical, symbol Connector:Conn_01x04_Female
- added R10, R13: ???20k, Resistor_SMD:R_0805_2012Metric_Pad1.20x1.40mm_HandSolder, symbol Device:R_Small
- added R11, R14: ???100k, Resistor_SMD:R_0805_2012Metric_Pad1.20x1.40mm_HandSolder, symbol Device:R_Small
- added R12, R15: 2.2k, Resistor_SMD:R_0805_2012Metric_Pad1.20x1.40mm_HandSolder, symbol Device:R_Small
- added SW3, SW4: SW_Push, Button_Switch_Keyboard:SW_Cherry_MX_1.00u_Plate, symbol Switch:SW_Push
- added unit 3 of U1
- added unit 4 of U1
- D1, D2: footprint Diode_THT:D_DO-41_SOD81_P7.62mm_Horizontal -> Diode_THT:D_DO-35_SOD27_P7.62mm_Horizontal
- R1: renamed from R4; footprint Resistor_THT:R_Axial_DIN0204_L3.6mm_D1.6mm_P2.54mm_Vertical -> Resistor_SMD:R_0805_2012Metric_Pad1.20x1.40mm_HandSolder
- R2: renamed from R5; footprint Resistor_THT:R_Axial_DIN0204_L3.6mm_D1.6mm_P2.54mm_Vertical -> Resistor_SMD:R_0805_2012Metric_Pad1.20x1.40mm_HandSolder
- R3: renamed from R7; footprint Resistor_THT:R_Axial_DIN0204_L3.6mm_D1.6mm_P2.54mm_Vertical -> Resistor_SMD:R_0805_2012Metric_Pad1.20x1.40mm_HandSolder
- R6: renamed from R8; footprint Resistor_THT:R_Axial_DIN0204_L3.6mm_D1.6mm_P2.54mm_Vertical -> Resistor_SMD:R_0805_2012Metric_Pad1.20x1.40mm_HandSolder
- R7: renamed from R9; footprint Resistor_THT:R_Axial_DIN0204_L3.6mm_D1.6mm_P2.54mm_Vertical -> Resistor_SMD:R_0805_2012Metric_Pad1.20x1.40mm_HandSolder
- R9: renamed from R10; footprint Resistor_THT:R_Axial_DIN0204_L3.6mm_D1.6mm_P2.54mm_Vertical -> Resistor_SMD:R_0805_2012Metric_Pad1.20x1.40mm_HandSolder
- renumbered C4 to C3, C5 to C6, J2 to J1, J3 to J2, R1 to R4, R2 to R5, R3 to R8
Connections:
- net 5V_Ard: now also J3.1 (Pin_1), J5.1 (Pin_1), R10.1, R13.1
- net Butt1: now also A1.13 (D10), J7.1 (Pin_1), J8.1 (Pin_1); no longer A1.6 (D3)
- net Butt2: now also A1.12 (D9), J7.2 (Pin_2), J8.2 (Pin_2); no longer A1.9 (D6)
- net GND: now also C4.2, C5.2, J4.1 (Pin_1), J6.1 (Pin_1), SW3.1, SW4.1
- net Butt4: now reaches A1.10 (D7)
- net Butt4: now also J7.4 (Pin_4), J8.4 (Pin_4), U1.11
- net Led renamed Butt3
- net Butt3: now also J7.3 (Pin_3), J8.3 (Pin_3), U1.10
- new net: R10.2, R11.1, R12.1, SW3.2
- new net: C4.1, R11.2
- new net: R12.2, U1.8, U1.9
- new net: R13.2, R14.1, R15.1, SW4.2
- new net: C5.1, R14.2
- new net: R15.2, U1.12, U1.13
Other:
- moved on the sheet: C2, C3, C6, R1, R2, R3, R6, R7, R9, SW1, SW2, U1A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

Commit message: s
Parts:
- C2, C3, C4, C5: value 100nF???10nF -> 0.1uF
- R1, R10, R13, R6: value ???20k -> 10k
- R11, R14, R2, R7: value ???100k -> 68
Changed lines of the file:
@@
 P 1700 4700
 F 0 "R1" H 1759 4746 50  0000 L CNN
-F 1 "???20k" H 1759 4655 50  0000 L CNN
+F 1 "10k" H 1759 4655 50  0000 L CNN
 F 2 "Resistor_SMD:R_0805_2012Metric_Pad1.20x1.40mm_HandSolder" H 1700 4700 50  0001 C CNN
 F 3 "~" H 1700 4700 50  0001 C CNN
@@
 P 2250 5700
 F 0 "C2" H 2342 5746 50  0000 L CNN
-F 1 "100nF???10nF" H 2342 5655 50  0000 L CNN
+F 1 "0.1uF" H 2342 5655 50  0000 L CNN
 F 2 "Capacitor_SMD:C_0805_2012Metric_Pad1.18x1.45mm_HandSolder" H 2250 5700 50  0001 C CNN
 F 3 "~" H 2250 5700 50  0001 C CNN
@@
 P 2050 5500
 F 0 "R2" V 2250 5550 50  0000 L CNN
-F 1 "???100k" V 2150 5350 50  0000 L CNN
+F 1 "68" V 2150 5350 50  0000 L CNN
 F 2 "Resistor_SMD:R_0805_2012Metric_Pad1.20x1.40mm_HandSolder" H 2050 5500 50  0001 C CNN
 F 3 "~" H 2050 5500 50  0001 C CNN
@@
 P 4500 5500
 F 0 "R7" V 4700 5550 50  0000 L CNN
-F 1 "???100k" V 4600 5350 50  0000 L CNN
+F 1 "68" V 4600 5350 50  0000 L CNN
 F 2 "Resistor_SMD:R_0805_2012Metric_Pad1.20x1.40mm_HandSolder" H 4500 5500 50  0001 C CNN
 F 3 "~" H 4500 5500 50  0001 C CNN
@@
 P 4700 5700
 F 0 "C3" H 4792 5746 50  0000 L CNN
-F 1 "100nF???10nF" H 4792 5655 50  0000 L CNN
+F 1 "0.1uF" H 4792 5655 50  0000 L CNN
 F 2 "Capacitor_SMD:C_0805_2012Metric_Pad1.18x1.45mm_HandSolder" H 4700 5700 50  0001 C CNN
 F 3 "~" H 4700 5700 50  0001 C CNN
@@
 P 4150 4700
 F 0 "R6" H 4209 4746 50  0000 L CNN
-F 1 "???20k" H 4209 4655 50  0000 L CNN
+F 1 "10k" H 4209 4655 50  0000 L CNN
 F 2 "Resistor_SMD:R_0805_2012Metric_Pad1.20x1.40mm_HandSolder" H 4150 4700 50  0001 C CNN
 F 3 "~" H 4150 4700 50  0001 C CNN
@@
 P 6800 4600
 F 0 "R10" H 6859 4646 50  0000 L CNN
-F 1 "???20k" H 6859 4555 50  0000 L CNN
+F 1 "10k" H 6859 4555 50  0000 L CNN
 F 2 "Resistor_SMD:R_0805_2012Metric_Pad1.20x1.40mm_HandSolder" H 6800 4600 50  0001 C CNN
 F 3 "~" H 6800 4600 50  0001 C CNN
@@
 P 7350 5600
 F 0 "C4" H 7442 5646 50  0000 L CNN
-F 1 "100nF???10nF" H 7442 5555 50  0000 L CNN
+F 1 "0.1uF" H 7442 5555 50  0000 L CNN
 F 2 "Capacitor_SMD:C_0805_2012Metric_Pad1.18x1.45mm_HandSolder" H 7350 5600 50  0001 C CNN
 F 3 "~" H 7350 5600 50  0001 C CNN
@@
 P 7150 5400
 F 0 "R11" V 7350 5450 50  0000 L CNN
-F 1 "???100k" V 7250 5250 50  0000 L CNN
+F 1 "68" V 7250 5250 50  0000 L CNN
 F 2 "Resistor_SMD:R_0805_2012Metric_Pad1.20x1.40mm_HandSolder" H 7150 5400 50  0001 C CNN
 F 3 "~" H 7150 5400 50  0001 C CNN
@@
 P 9600 5400
 F 0 "R14" V 9800 5450 50  0000 L CNN
-F 1 "???100k" V 9700 5250 50  0000 L CNN
+F 1 "68" V 9700 5250 50  0000 L CNN
 F 2 "Resistor_SMD:R_0805_2012Metric_Pad1.20x1.40mm_HandSolder" H 9600 5400 50  0001 C CNN
 F 3 "~" H 9600 5400 50  0001 C CNN
@@
 P 9800 5600
 F 0 "C5" H 9892 5646 50  0000 L CNN
-F 1 "100nF???10nF" H 9892 5555 50  0000 L CNN
+F 1 "0.1uF" H 9892 5555 50  0000 L CNN
 F 2 "Capacitor_SMD:C_0805_2012Metric_Pad1.18x1.45mm_HandSolder" H 9800 5600 50  0001 C CNN
 F 3 "~" H 9800 5600 50  0001 C CNN
@@
 P 9250 4600
 F 0 "R13" H 9309 4646 50  0000 L CNN
-F 1 "???20k" H 9309 4555 50  0000 L CNN
+F 1 "10k" H 9309 4555 50  0000 L CNN
 F 2 "Resistor_SMD:R_0805_2012Metric_Pad1.20x1.40mm_HandSolder" H 9250 4600 50  0001 C CNN
 F 3 "~" H 9250 4600 50  0001 C CNN

Commit message: ы
Parts:
- removed R11, R14, R2, R7: 68, Resistor_SMD:R_0805_2012Metric_Pad1.20x1.40mm_HandSolder, symbol Device:R_Small
- R12, R15, R3, R9: value 2.2k -> 100k
Connections:
- net at R3.2, U1.1, U1.2: now also C2.1
- net at R9.2, U1.5, U1.6: now also C3.1
- net at C4.1: now also R12.2, U1.8, U1.9
- net at C5.1: now also R15.2, U1.12, U1.13
Other:
- moved on the sheet: C2, C3, C4, C5
Changed lines of the file:
@@
 L Device:C_Small C2
 U 1 1 61883E27
-P 2250 5700
-F 0 "C2" H 2342 5746 50  0000 L CNN
-F 1 "0.1uF" H 2342 5655 50  0000 L CNN
-F 2 "Capacitor_SMD:C_0805_2012Metric_Pad1.18x1.45mm_HandSolder" H 2250 5700 50  0001 C CNN
-F 3 "~" H 2250 5700 50  0001 C CNN
-	1    2250 5700
+P 2400 5550
+F 0 "C2" H 2492 5596 50  0000 L CNN
+F 1 "0.1uF" H 2492 5505 50  0000 L CNN
+F 2 "Capacitor_SMD:C_0805_2012Metric_Pad1.18x1.45mm_HandSolder" H 2400 5550 50  0001 C CNN
+F 3 "~" H 2400 5550 50  0001 C CNN
+	1    2400 5550
 	1    0    0    -1
 $EndComp
@@
 	1550 5500 1700 5500
 Wire Wire Line
-	1550 5900 1550 6200
-Connection ~ 1550 5900
+	1550 5900 1550 6050
 $Comp
 L Device:R_Small R3
 U 1 1 61883E36
 P 2250 5150
-F 0 "R3" V 2450 5200 50  0000 L CNN
-F 1 "2.2k" V 2350 5000 50  0000 L CNN
+F 0 "R3" V 2450 5150 50  0000 L CNN
+F 1 "100k" V 2350 5050 50  0000 L CNN
 F 2 "Resistor_SMD:R_0805_2012Metric_Pad1.20x1.40mm_HandSolder" H 2250 5150 50  0001 C CNN
 F 3 "~" H 2250 5150 50  0001 C CNN
@@
 $EndComp
 Wire Wire Line
-	2350 5150 2550 5150
+	2350 5150 2400 5150
 Connection ~ 2550 5150
 Wire Wire Line
@@
 	1700 5150 1700 5500
 Connection ~ 1700 5150
-Connection ~ 1700 5500
-Wire Wire Line
-	1700 5500 1950 5500
 Wire Wire Line
 	3300 5250 3200 5250
 Wire Wire Line
 	2600 5350 2550 5350
-$Comp
-L Device:R_Small R2
-U 1 1 61883E48
-P 2050 5500
-F 0 "R2" V 2250 5550 50  0000 L CNN
-F 1 "68" V 2150 5350 50  0000 L CNN
-F 2 "Resistor_SMD:R_0805_2012Metric_Pad1.20x1.40mm_HandSolder" H 2050 5500 50  0001 C CNN
-F 3 "~" H 2050 5500 50  0001 C CNN
-	1    2050 5500
-	0    -1   -1   0
-$EndComp
-Wire Wire Line
-	2150 5500 2250 5500
-Wire Wire Line
-	2250 5500 2250 5600
-Wire Wire Line
-	2250 5800 2250 5900
-Wire Wire Line
-	1550 5900 2250 5900
-Wire Wire Line
-	4000 5900 4700 5900
-Wire Wire Line
-	4700 5800 4700 5900
-Wire Wire Line
-	4700 5500 4700 5600
-Wire Wire Line
-	4600 5500 4700 5500
-$Comp
-L Device:R_Small R7
-U 1 1 618787F3
-P 4500 5500
-F 0 "R7" V 4700 5550 50  0000 L CNN
-F 1 "68" V 4600 5350 50  0000 L CNN
-F 2 "Resistor_SMD:R_0805_2012Metric_Pad1.20x1.40mm_HandSolder" H 4500 5500 50  0001 C CNN
-F 3 "~" H 4500 5500 50  0001 C CNN
-	1    4500 5500
-	0    -1   -1   0
-$EndComp
 Wire Wire Line
 	5050 5350 5000 5350
@@
 Text Label 800  2800 2    50   ~ 0
 Butt3
-Wire Wire Line
-	4150 5500 4400 5500
-Connection ~ 4150 5500
 Connection ~ 4150 5150
 Wire Wire Line
@@
 Connection ~ 5000 5150
 Wire Wire Line
-	4800 5150 5000 5150
-$Comp
-L Device:R_Small R9
-U 1 1 6186E060
-P 4700 5150
-F 0 "R9" V 4900 5200 50  0000 L CNN
-F 1 "2.2k" V 4800 5000 50  0000 L CNN
-F 2 "Resistor_SMD:R_0805_2012Metric_Pad1.20x1.40mm_HandSolder" H 4700 5150 50  0001 C CNN
-F 3 "~" H 4700 5150 50  0001 C CNN
-	1    4700 5150
-	0    -1   -1   0
-$EndComp
+	4800 5150 4850 5150
 Connection ~ 4000 5900
 Wire Wire Line
@@
 L Device:C_Small C3
 U 1 1 6186E04E
-P 4700 5700
-F 0 "C3" H 4792 5746 50  0000 L CNN
-F 1 "0.1uF" H 4792 5655 50  0000 L CNN
-F 2 "Capacitor_SMD:C_0805_2012Metric_Pad1.18x1.45mm_HandSolder" H 4700 5700 50  0001 C CNN
-F 3 "~" H 4700 5700 50  0001 C CNN
-	1    4700 5700
+P 4850 5500
+F 0 "C3" H 4942 5546 50  0000 L CNN
+F 1 "0.1uF" H 4942 5455 50  0000 L CNN
+F 2 "Capacitor_SMD:C_0805_2012Metric_Pad1.18x1.45mm_HandSolder" H 4850 5500 50  0001 C CNN
+F 3 "~" H 4850 5500 50  0001 C CNN
+	1    4850 5500
 	1    0    0    -1
 $EndComp
@@
 L Device:C_Small C4
 U 1 1 6198DCED
-P 7350 5600
-F 0 "C4" H 7442 5646 50  0000 L CNN
-F 1 "0.1uF" H 7442 5555 50  0000 L CNN
-F 2 "Capacitor_SMD:C_0805_2012Metric_Pad1.18x1.45mm_HandSolder" H 7350 5600 50  0001 C CNN
-F 3 "~" H 7350 5600 50  0001 C CNN
-	1    7350 5600
+P 7500 5400
+F 0 "C4" H 7592 5446 50  0000 L CNN
+F 1 "0.1uF" H 7592 5355 50  0000 L CNN
+F 2 "Capacitor_SMD:C_0805_2012Metric_Pad1.18x1.45mm_HandSolder" H 7500 5400 50  0001 C CNN
+F 3 "~" H 7500 5400 50  0001 C CNN
+	1    7500 5400
 	1    0    0    -1
 $EndComp
@@
 U 1 1 6198DCFC
 P 7350 5050
-F 0 "R12" V 7550 5100 50  0000 L CNN
-F 1 "2.2k" V 7450 4900 50  0000 L CNN
+F 0 "R12" V 7550 5050 50  0000 L CNN
+F 1 "100k" V 7450 5000 50  0000 L CNN
 F 2 "Resistor_SMD:R_0805_2012Metric_Pad1.20x1.40mm_HandSolder" H 7350 5050 50  0001 C CNN
 F 3 "~" H 7350 5050 50  0001 C CNN
@@
 $EndComp
 Wire Wire Line
-	7450 5050 7650 5050
+	7450 5050 7500 5050
 Connection ~ 7650 5050
 Wire Wire Line
@@
 	6800 5050 6800 5400
 Connection ~ 6800 5050
-Connection ~ 6800 5400
-Wire Wire Line
-	6800 5400 7050 5400
 Wire Wire Line
 	8400 5150 8300 5150
 Wire Wire Line
 	7700 5250 7650 5250
-$Comp
-L Device:R_Small R11
-U 1 1 6198DD0D
-P 7150 5400
-F 0 "R11" V 7350 5450 50  0000 L CNN
-F 1 "68" V 7250 5250 50  0000 L CNN
-F 2 "Resistor_SMD:R_0805_2012Metric_Pad1.20x1.40mm_HandSolder" H 7150 5400 50  0001 C CNN
-F 3 "~" H 7150 5400 50  0001 C CNN
-	1    7150 5400
-	0    -1   -1   0
-$EndComp
-Wire Wire Line
-	7250 5400 7350 5400
-Wire Wire Line
-	7350 5400 7350 5500
-Wire Wire Line
-	7350 5700 7350 5800
-Wire Wire Line
-	6650 5800 7350 5800
-Wire Wire Line
-	9100 5800 9800 5800
-Wire Wire Line
-	9800 5700 9800 5800
-Wire Wire Line
-	9800 5400 9800 5500
-Wire Wire Line
-	9700 5400 9800 5400
-$Comp
-L Device:R_Small R14
-U 1 1 6198DD1B
-P 9600 5400
-F 0 "R14" V 9800 5450 50  0000 L CNN
-F 1 "68" V 9700 5250 50  0000 L CNN
-F 2 "Resistor_SMD:R_0805_2012Metric_Pad1.20x1.40mm_HandSolder" H 9600 5400 50  0001 C CNN
-F 3 "~" H 9600 5400 50  0001 C CNN
-	1    9600 5400
-	0    -1   -1   0
-$EndComp
 Wire Wire Line
 	10150 5250 10100 5250
 Wire Wire Line
 	10850 5150 10750 5150
-Wire Wire Line
-	9250 5400 9500 5400
-Connection ~ 9250 5400
 Connection ~ 9250 5050
 Wire Wire Line
@@
 Connection ~ 10100 5050
 Wire Wire Line
-	9900 5050 10100 5050
+	9900 5050 10000 5050
 $Comp
 L Device:R_Small R15
 U 1 1 6198DD2C
 P 9800 5050
-F 0 "R15" V 10000 5100 50  0000 L CNN
-F 1 "2.2k" V 9900 4900 50  0000 L CNN
+F 0 "R15" V 10000 5000 50  0000 L CNN
+F 1 "100k" V 9900 5000 50  0000 L CNN
 F 2 "Resistor_SMD:R_0805_2012Metric_Pad1.20x1.40mm_HandSolder" H 9800 5050 50  0001 C CNN
 F 3 "~" H 9800 5050 50  0001 C CNN
@@
 Wire Wire Line
 	9100 5400 9250 5400
-$Comp
-L Device:C_Small C5
-U 1 1 6198DD3B
-P 9800 5600
-F 0 "C5" H 9892 5646 50  0000 L CNN
-F 1 "0.1uF" H 9892 5555 50  0000 L CNN
-F 2 "Capacitor_SMD:C_0805_2012Metric_Pad1.18x1.45mm_HandSolder" H 9800 5600 50  0001 C CNN
-F 3 "~" H 9800 5600 50  0001 C CNN
-	1    9800 5600
-	1    0    0    -1
-$EndComp
 Wire Wire Line
 	10100 5050 10100 5250
@@
 Wire Wire Line
 	4650 3050 5050 3050
+Wire Wire Line
+	2400 5150 2400 5450
+Connection ~ 2400 5150
+Wire Wire Line
+	2400 5150 2550 5150
+Wire Wire Line
+	2400 5650 2400 6050
+Wire Wire Line
+	2400 6050 1550 6050
+Connection ~ 1550 6050
+Wire Wire Line
+	1550 6050 1550 6200
+$Comp
+L Device:R_Small R9
+U 1 1 6186E060
+P 4700 5150
+F 0 "R9" V 4900 5200 50  0000 L CNN
+F 1 "100k" V 4800 5150 50  0000 L CNN
+F 2 "Resistor_SMD:R_0805_2012Metric_Pad1.20x1.40mm_HandSolder" H 4700 5150 50  0001 C CNN
+F 3 "~" H 4700 5150 50  0001 C CNN
+	1    4700 5150
+	0    -1   -1   0
+$EndComp
+Wire Wire Line
+	4850 5400 4850 5150
+Connection ~ 4850 5150
+Wire Wire Line
+	4850 5150 5000 5150
+Wire Wire Line
+	4850 5600 4850 5900
+Wire Wire Line
+	4000 5900 4850 5900
+Wire Wire Line
+	7500 5300 7500 5050
+Connection ~ 7500 5050
+Wire Wire Line
+	7500 5050 7650 5050
+Wire Wire Line
+	7500 5500 7500 5800
+Wire Wire Line
+	6650 5800 7500 5800
+$Comp
+L Device:C_Small C5
+U 1 1 6198DD3B
+P 10000 5400
+F 0 "C5" H 10092 5446 50  0000 L CNN
+F 1 "0.1uF" H 10092 5355 50  0000 L CNN
+F 2 "Capacitor_SMD:C_0805_2012Metric_Pad1.18x1.45mm_HandSolder" H 10000 5400 50  0001 C CNN
+F 3 "~" H 10000 5400 50  0001 C CNN
+	1    10000 5400
+	1    0    0    -1
+$EndComp
+Wire Wire Line
+	10000 5300 10000 5050
+Connection ~ 10000 5050
+Wire Wire Line
+	10000 5050 10100 5050
+Wire Wire Line
+	10000 5500 10000 5800
+Wire Wire Line
+	9100 5800 10000 5800
 $EndSCHEMATC

Commit message: s
Parts:
- added Q1: AO3401A, Package_TO_SOT_SMD:SOT-23, symbol Transistor_FET:AO3401A
- added R2, R7: 2.2k, Resistor_SMD:R_0805_2012Metric_Pad1.20x1.40mm_HandSolder, symbol Device:R_Small
Connections:
- net 5V_Ard: now also Q1.3 (D); no longer A1.27 (+5V)
- net Keyboard_en: now reaches A1.6 (D3)
- net Keyboard_en: now also R2.2
- new net: A1.27 (+5V), Q1.2 (S), R7.1
- new net: Q1.1 (G), R2.1, R7.2
- no-connect marks 19 -> 18
Changed lines of the file:
@@
 	1    0    0    -1
 $EndComp
-Wire Wire Line
-	2100 1500 2050 1500
 $Comp
 L Device:C_Small C1
@@
 NoConn ~ 1950 1600
 Wire Wire Line
-	2050 1500 2050 1600
-Wire Wire Line
 	1750 1250 1750 1600
 $Comp
@@
 NoConn ~ 1350 2000
 NoConn ~ 1350 2100
-NoConn ~ 1350 2300
 Text Label 3900 4400 2    50   ~ 0
 5V_Conn
@@
 Text Label 10200 850  2    50   ~ 0
 5V_Conn
-Text Label 2100 1500 0    50   ~ 0
+Text Label 3500 2550 0    50   ~ 0
 5V_Ard
 Text Label 4750 2900 0    50   ~ 0
@@
 Wire Wire Line
 	9100 5800 10000 5800
+$Comp
+L Transistor_FET:AO3401A Q1
+U 1 1 61AD9259
+P 3300 2200
+F 0 "Q1" H 3505 2154 50  0000 L CNN
+F 1 "AO3401A" H 3505 2245 50  0000 L CNN
+F 2 "Package_TO_SOT_SMD:SOT-23" H 3500 2125 50  0001 L CIN
+F 3 "http://www.aosmd.com/pdfs/datasheet/AO3401A.pdf" H 3300 2200 50  0001 L CNN
+	1    3300 2200
+	1    0    0    1
+$EndComp
+Wire Wire Line
+	3400 2550 3400 2400
+$Comp
+L Device:R_Small R7
+U 1 1 61AED0AD
+P 3000 1950
+F 0 "R7" H 3059 1996 50  0000 L CNN
+F 1 "2.2k" H 3059 1905 50  0000 L CNN
+F 2 "Resistor_SMD:R_0805_2012Metric_Pad1.20x1.40mm_HandSolder" H 3000 1950 50  0001 C CNN
+F 3 "~" H 3000 1950 50  0001 C CNN
+	1    3000 1950
+	1    0    0    -1
+$EndComp
+Wire Wire Line
+	3100 2200 3000 2200
+Wire Wire Line
+	2050 1600 2900 1600
+Wire Wire Line
+	2900 1600 2900 1800
+Text Label 2950 2600 2    50   ~ 0
+Keyboard_en
+Wire Wire Line
+	2950 2300 2950 2200
+Wire Wire Line
+	2950 2200 3000 2200
+Connection ~ 3000 2200
+$Comp
+L Device:R_Small R2
+U 1 1 61B0FCFB
+P 2950 2400
+F 0 "R2" H 3009 2446 50  0000 L CNN
+F 1 "2.2k" H 3009 2355 50  0000 L CNN
+F 2 "Resistor_SMD:R_0805_2012Metric_Pad1.20x1.40mm_HandSolder" H 2950 2400 50  0001 C CNN
+F 3 "~" H 2950 2400 50  0001 C CNN
+	1    2950 2400
+	1    0    0    -1
+$EndComp
+Wire Wire Line
+	2900 1800 3000 1800
+Wire Wire Line
+	3000 1850 3000 1800
+Connection ~ 3000 1800
+Wire Wire Line
+	3000 1800 3400 1800
+Wire Wire Line
+	3000 2050 3000 2200
+Wire Wire Line
+	3400 1800 3400 2000
+Wire Wire Line
+	2950 2500 2950 2600
+Wire Wire Line
+	3500 2550 3400 2550
+Text Label 1050 2300 2    50   ~ 0
+Keyboard_en
+Wire Wire Line
+	1050 2300 1350 2300
 $EndSCHEMATC
