File: !Kursach/LX/lx_switch/sw/sw.sch (KiCad schematic (older format))
At the start: 6 parts, among them J1 bat, J2 usb, J3 out, Q1 AO3401A

Commit message: fuck
Parts:
- added VD?: VD_SCHOTTKY, symbol Diodes:VD_SCHOTTKY
- added VT?: VT_PMOS_ENH_GSD, symbol Transistors:VT_PMOS_ENH_GSD
Changed lines of the file:
@@
 Wire Wire Line
 	4700 2000 4700 1950
+$Comp
+L Transistors:VT_PMOS_ENH_GSD VT?
+U 1 1 61AD3AD1
+P 3800 3300
+F 0 "VT?" H 4088 3361 70  0000 L CNN
+F 1 "VT_PMOS_ENH_GSD" H 4088 3240 70  0000 L CNN
+F 2 "" H 3800 3300 70  0001 C CNN
+F 3 "" H 3800 3300 70  0001 C CNN
+	1    3800 3300
+	1    0    0    -1
+$EndComp
+$Comp
+L Diodes:VD_SCHOTTKY VD?
+U 1 1 61AD6403
+P 3150 3800
+F 0 "VD?" H 3444 3861 70  0000 L CNN
+F 1 "VD_SCHOTTKY" H 3444 3740 70  0000 L CNN
+F 2 "" H 3150 3800 70  0001 C CNN
+F 3 "" H 3150 3800 70  0001 C CNN
+	1    3150 3800
+	0    1    1    0
+$EndComp
 $EndSCHEMATC
